File: cc-ring.kicad_pcb (KiCad board)
At the start: 2 copper layers, 75 x 5.5 mm, 40 parts, among them J1 Battery, J2 Debug, J3 Battery, J4 Charge, U1 STM32L431CCYx, U2 BQ297xy, U3 CSD83325L

Commit message: make it manufacturable lol
Parts:
- removed D10: D_Small, Diode_SMD:D_SOD-523
- removed R1: 1M, Resistor_SMD:R_0402_1005Metric
- added C14: 100n, Capacitor_SMD:C_0402_1005Metric, B.Cu at (179.6, 71.0)
- added C15: 100n, Capacitor_SMD:C_0402_1005Metric, B.Cu at (177.1, 70.0)
- added G***: LOGO, pretzel:pretzel, F.Cu at (235.3, 71.0)
- added U4: TLV70736DQNR, tlv707:DQN0004A, B.Cu at (178.3, 70.6)
- moved D9 1.58 mm to (177.4, 72.2), turned to 180 degrees
- moved C6 0.08 mm to (178.5, 69.1)
Connections:
- J1 pad 2: -BATT -> -BATT2
- J3 pad 1: -BATT -> -BATT2
- U3 pad C1: -BATT -> -BATT2
Routing:
- net +BATT: track 92.0 -> 24.8 mm
- net -BATT: track 9.41 -> 2.66 mm, vias 2 -> 1
- net -BATT2: track 0.00 -> 4.21 mm, vias 0 -> 1
- net Net-(D1-DOUT): track 2.63 -> 6.40 mm
- net Net-(D2-DOUT): track 2.63 -> 6.06 mm
- net Net-(D5-DOUT): track 2.63 -> 5.90 mm
- net Net-(D7-DOUT): track 2.63 -> 5.81 mm
- net Net-(D3-DOUT): track 2.63 -> 5.55 mm
- net Net-(D15-DOUT): track 2.63 -> 5.48 mm
- net Net-(D11-DOUT): track 2.63 -> 5.42 mm
- net Net-(D13-DOUT): track 2.63 -> 5.38 mm
- net LED_SNS: track 4.36 -> 2.05 mm
- net Net-(U2-Cout): track 3.09 -> 5.29 mm, vias 0 -> 2
- net GND: track 11.9 -> 11.2 mm, vias 32 -> 50
- added copper zone on B.Cu, net +BATT
Other:
- rule pad_to_mask_clearance: 0 -> 0.1
- board text added: "JL"
- board text added: "LED Ring v0.2"
- board text added: "Nov 2024"
